File: circuit/circuit.kicad_sch (KiCad schematic)
At the start: 25 parts, among them M1 Stepper, M2 Stepper

Commit message: changes to circuit
Parts:
- removed BT?: 7.2V NiMH, symbol Device:Battery_Cell
- added U?: LM2595_Module, symbol Regulator_Switching:LM2595_Module
Connections:
- net +5V: now also U?. (OUT-); no longer A?.5 (+5V)
- net +BATT: now also U?. (OUT-)
- net GND: now also U?. (OUT-)
- net NC: now also A?.5 (+5V)
Other:
- moved on the sheet: BT?
